File: plan/RF.kicad_sch (KiCad schematic)
At the start: 0 parts

Commit message: Assign footprints to devices on power schematic
Parts:
- added AE1: 2450AT18A0100001E, Smarthome:Antenna_Johanson_2450AT18A0100001E, symbol Smarthome:Johanson_2450AT18A0100001E
- added C1: 2,3 pF, Capacitor_SMD:C_0201_0603Metric, symbol Device:C
- added C2: 1,6 pF, Capacitor_SMD:C_0201_0603Metric, symbol Device:C
- added C3: 0,3 pF, Capacitor_SMD:C_0201_0603Metric, symbol Device:C
- added C4, C5: TUNE, Capacitor_SMD:C_0201_0603Metric, symbol Device:C
- added CC1: 0 Ω, Resistor_SMD:R_0201_0603Metric, symbol Device:R
- added L1: 2,9 nH, Inductor_SMD:L_0201_0603Metric, symbol Device:L
- added L2: 1,2 nH, Inductor_SMD:L_0201_0603Metric, symbol Device:L
- added L3: TUNE, Inductor_SMD:L_0201_0603Metric, symbol Device:L
Connections:
- new net: C2.1, L1.2, L2.1
- new net: C3.1, CC1.1, L2.2
- new net: AE1.1 (FEED), C5.1, L3.2
- new net GND: C1.2, C2.2, C3.2, C4.2, C5.2
- new net RF2G4_IO: C1.1, L1.1
- new net RF_50OHM: C4.1, CC1.2, L3.1
Other:
- note added: "Silicon-Labs-MG24-Matching/Harmonic-Filter"
- note added: "π-Matching-Network Johanson Antenna"
