File: plan/MCU.kicad_sch (KiCad schematic)
At the start: 0 parts

Commit message: Create MCU schematic according to datasheet of MG24 and reference design
Parts:
- added U1: EFR32MG24B020F1536IM48-B, Smarthome:QFN-48-1EP_6x6mm_P0.4mm_EFR32MG24, symbol Smarthome:EFR32MG24B020F1536IM48-B
- added Y1: XTL501250-S315-038, Smarthome:Crystal_Siward_XTL501250_2.0x1.6mm, symbol Smarthome:Siward_XTL501250
Connections:
- new net: U1.11 (HFXTAL_I), Y1.1
- new net: U1.12 (HFXTAL_O), Y1.3
- new net AVDD: U1.41 (AVDD)
- new net DECOUPLE: U1.36 (DECOUPLE)
- new net DVDD: U1.40 (DVDD)
- new net GND: U1.15 (RFVSS), U1.39 (VREGVSS), U1.49 (VSS), Y1.2 (G), Y1.4 (G)
- new net IOVDD: U1.42 (IOVDD)
- new net PA00: U1.26 (PA00)
- new net PA01: U1.27 (PA01)
- new net PA02: U1.28 (PA02)
- new net PA03: U1.29 (PA03)
- new net PA04: U1.30 (PA04)
- new net PA05: U1.31 (PA05)
- new net PA06: U1.32 (PA06)
- new net PA07: U1.33 (PA07)
- new net PA08: U1.34 (PA08)
- new net PA09: U1.35 (PA09)
- new net PAVDD: U1.17 (PAVDD)
- new net PB00: U1.23 (PB00)
- new net PB01: U1.22 (PB01)
- new net PB02: U1.21 (PB02)
- new net PB03: U1.20 (PB03)
- new net PB04: U1.19 (PB04)
- new net PB05: U1.18 (PB05)
- new net PC00: U1.1 (PC00)
- new net PC01: U1.2 (PC01)
- new net PC02: U1.3 (PC02)
- new net PC03: U1.4 (PC03)
- new net PC04: U1.5 (PC04)
- new net PC05: U1.6 (PC05)
- new net PC06: U1.7 (PC06)
- new net PC07: U1.8 (PC07)
- new net PC08: U1.9 (PC08)
- new net PC09: U1.10 (PC09)
- new net PD00: U1.48 (PD00)
- new net PD01: U1.47 (PD01)
- new net PD02: U1.46 (PD02)
- new net PD03: U1.45 (PD03)
- new net PD04: U1.44 (PD04)
- new net PD05: U1.43 (PD05)
- new net RF2G4_IO: U1.16 (RF2G4_IO)
- new net RFVDD: U1.14 (RFVDD)
- new net VREGSW: U1.37 (VREGSW)
- new net VREGVDD: U1.38 (VREGVDD)
- new net ~{RESET}: U1.13 (~{RESET})
- no-connect marks 0 -> 2
Other:
- note added: "not connected"

Commit message: Adapt schematics to pass ERC
- Clean AVDD / IOVDD / VREGVDD: use VBAT instead
- Clean DVDD / VDCDC: remove net DVDD and use VDCDC instead
- Use original symbol from library for J1
- Mark VBAT / VDCDC / RFVDD / PAVDD / GND with PWR_FLAG
Connections:
- net IOVDD is gone; now on net VBAT: U1.42 (IOVDD)
- net VREGVDD is gone; now on net VBAT: U1.38 (VREGVDD)
- net AVDD renamed VBAT
- net DVDD renamed VDCDC
Changed lines of the file:
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@@
 		)
 	)
-	(global_label "DVDD"
+	(global_label "VDCDC"
 		(shape input)
 		(at 165.1 57.15 0)
@@
 		)
 		(property "Intersheetrefs" "${INTERSHEET_REFS}"
-			(at 172.9838 57.15 0)
+			(at 174.2538 57.15 0)
 			(hide yes)
 			(show_name no)
@@
 		)
 	)
-	(global_label "AVDD"
+	(global_label "VBAT"
 		(shape input)
 		(at 177.8 54.61 0)
@@
 		)
 		(property "Intersheetrefs" "${INTERSHEET_REFS}"
-			(at 185.5024 54.61 0)
-			(hide yes)
-			(show_name no)
-			(do_not_autoplace no)
-			(effects
-				(font
-					(size 1.27 1.27)
-				)
-				(justify left)
-			)
-		)
-	)
-	(global_label "IOVDD"
+			(at 185.2 54.61 0)
+			(hide yes)
+			(show_name no)
+			(do_not_autoplace no)
+			(effects
+				(font
+					(size 1.27 1.27)
+				)
+				(justify left)
+			)
+		)
+	)
+	(global_label "VBAT"
 		(shape input)
 		(at 177.8 59.69 0)
@@
 		)
 		(property "Intersheetrefs" "${INTERSHEET_REFS}"
-			(at 186.3491 59.69 0)
+			(at 185.2 59.69 0)
 			(hide yes)
 			(show_name no)
@@
 		)
 	)
-	(global_label "VREGVDD"
+	(global_label "VBAT"
 		(shape input)
 		(at 165.1 52.07 0)
@@
 		)
 		(property "Intersheetrefs" "${INTERSHEET_REFS}"
-			(at 176.4914 52.07 0)
-			(hide yes)
-			(show_name no)
+			(at 172.5 52.07 0)
+			(hide yes)
+			(show_name no)
