File: plan/Power.kicad_sch (KiCad schematic)
At the start: 0 parts

Commit message: Create power schematic according to datasheet of MG24 and reference design
Parts:
- added C101, C111, C112: 100 nF, symbol Device:C
- added C102: 10 µF, symbol Device:C_Polarized
- added C103: 4,7 µF, symbol Device:C_Polarized
- added C104, C105, C106, C109, C110: 1 µF, symbol Device:C_Polarized
- added C107: 18 pF, symbol Device:C
- added C108: 0,5 pF, symbol Device:C
- added FB101: 70 Ω @ 100 MHz, symbol Device:FerriteBead_Small
- added L101: 2,2 µH, symbol Device:L
- added R101, R102: 0 Ω, symbol Device:R
Connections:
- new net AVDD: C101.1, C102.1, C109.1, C110.1, C111.1, C112.1, R101.1
- new net DECOUPLE: C104.1
- new net DVDD: C103.1, FB101.1, L101.2, R102.1
- new net GND: C101.2, C102.2, C103.2, C104.2, C105.2, C106.2, C107.2, C108.2, C109.2, C110.2, C111.2, C112.2
- new net PAVDD: C106.1, C107.1, C108.1, R101.2, R102.2
- new net RFVDD: C105.1, FB101.2
- new net VREGSW: L101.1
Other:
- note added: "PAVDD source select - populate only R101 or R102"

Commit message: Assign footprints to devices on power schematic
Parts:
- C101, C104, C105, C106, C109, C110, C111, C112: footprint (none) -> Capacitor_SMD:C_0402_1005Metric
- C102, C103: footprint (none) -> Capacitor_SMD:C_0603_1608Metric
- C107, C108: footprint (none) -> Capacitor_SMD:C_0201_0603Metric
- FB101: footprint (none) -> Inductor_SMD:L_0201_0603Metric
- L101: value 2,2 µH -> DFE2HCAH2R2MJ0; footprint (none) -> Smarthome:Inductor_Murata_DFE2HCAH_2520; symbol Device:L -> Smarthome:DFE2HCAH2R2MJ0; MPN (none) -> DFE2HCAH2R2MJ0; Manufacturer (none) -> Murata Electronics
- R101, R102: footprint (none) -> Resistor_SMD:R_0402_1005Metric
Changed lines of the file:
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@@
 			)
 		)
-		(property "Footprint" ""
+		(property "Footprint" "Capacitor_SMD:C_0603_1608Metric"
 			(at 155.9052 74.93 0)
 			(hide yes)
@@
 	)
 	(symbol
-		(lib_id "Device:L")
+		(lib_id "Smarthome:DFE2HCAH2R2MJ0")
 		(at 146.05 60.96 90)
 		(unit 1)
@@
 			)
 		)
-		(property "Value" "2,2 µH"
+		(property "Value" "DFE2HCAH2R2MJ0"
 			(at 146.05 58.42 90)
 			(show_name no)
@@
 			)
 		)
-		(property "Footprint" ""
+		(property "Footprint" "Smarthome:Inductor_Murata_DFE2HCAH_2520"
 			(at 146.05 60.96 0)
 			(hide yes)
@@
 			)
 		)
-		(property "Datasheet" ""
+		(property "Datasheet" "https://pim.murata.com/asset/pim4/inductor/JETE243A-9105_PDF_INDUCTOR?lastModifiedDatetime=20250708072123"
 			(at 146.05 60.96 0)
 			(hide yes)
@@
 			)
 		)
-		(property "Description" "Murata DFE2HCAH2R2MJ0"
+		(property "Description" "Murata DFE2HCAH power inductor, 2.2 µH, 2520 (1008), 2.5 x 2.0 x 1.2 mm"
+			(at 146.05 60.96 0)
+			(hide yes)
+			(show_name no)
+			(do_not_autoplace no)
+			(effects
+				(font
+					(size 1.27 1.27)
+				)
+			)
+		)
+		(property "Manufacturer" "Murata Electronics"
+			(at 146.05 60.96 0)
+			(hide yes)
+			(show_name no)
+			(do_not_autoplace no)
+			(effects
+				(font
+					(size 1.27 1.27)
+				)
+			)
+		)
+		(property "MPN" "DFE2HCAH2R2MJ0"
 			(at 146.05 60.96 0)
 			(hide yes)
@@
 			)
 		)
-		(property "Footprint" ""
+		(property "Footprint" "Capacitor_SMD:C_0603_1608Metric"
 			(at 75.8952 74.93 0)
 			(hide yes)
@@
 			)
 		)
-		(property "Footprint" ""
+		(property "Footprint" "Capacitor_SMD:C_0402_1005Metric"
 			(at 229.5652 125.73 0)
 			(hide yes)
@@
 			)
 		)
-		(property "Footprint" ""
+		(property "Footprint" "Capacitor_SMD:C_0201_0603Metric"
 			(at 144.4752 125.73 0)
 			(hide yes)
@@
 			)
 		)
-		(property "Footprint" ""
+		(property "Footprint" "Capacitor_SMD:C_0402_1005Metric"
 			(at 56.8452 74.93 0)
 			(hide yes)
@@
 			)
 		)
-		(property "Footprint" ""
+		(property "Footprint" "Capacitor_SMD:C_0201_0603Metric"
 			(at 130.5052 125.73 0)
 			(hide yes)
@@
 			)
 		)
-		(property "Footprint" ""
+		(property "Footprint" "Inductor_SMD:L_0201_0603Metric"
 			(at 232.41 62.738 90)
 			(hide yes)
@@
 			)
 		)
-		(property "Footprint" ""
+		(property "Footprint" "Capacitor_SMD:C_0402_1005Metric"
 			(at 178.7652 125.73 0)
 			(hide yes)
@@
 			)
 		)
-		(property "Footprint" ""
+		(property "Footprint" "Resistor_SMD:R_0402_1005Metric"
 			(at 60.96 137.668 90)
 			(hide yes)
@@
 			)
 		)
-		(property "Footprint" ""
+		(property "Footprint" "Capacitor_SMD:C_0402_1005Metric"
 			(at 194.0052 74.93 0)
 			(hide yes)
@@
 			)
 		)
-		(property "Footprint" ""
+		(property "Footprint" "Capacitor_SMD:C_0402_1005Metric"
 			(at 216.8652 125.73 0)
 			(hide yes)
@@
 			)
 		)
-		(property "Footprint" ""
+		(property "Footprint" "Resistor_SMD:R_0402_1005Metric"
 			(at 60.96 112.268 90)
 			(hide yes)
@@
 			)
 		)
-		(property "Footprint" ""
+		(property "Footprint" "Capacitor_SMD:C_0402_1005Metric"
 			(at 243.5352 74.93 0)
 			(hide yes)
@@
 			)
 		)
-		(property "Footprint" ""
+		(property "Footprint" "Capacitor_SMD:C_0402_1005Metric"
 			(at 115.2652 125.73 0)
 			(hide yes)
@@
 			)
 		)
-		(property "Footprint" ""
+		(property "Footprint" "Capacitor_SMD:C_0402_1005Metric"
 			(at 192.7352 125.73 0)
 			(hide yes)

Commit message: Adapt schematics to pass ERC
- Clean AVDD / IOVDD / VREGVDD: use VBAT instead
- Clean DVDD / VDCDC: remove net DVDD and use VDCDC instead
- Use original symbol from library for J1
- Mark VBAT / VDCDC / RFVDD / PAVDD / GND with PWR_FLAG
Connections:
- net AVDD renamed VBAT
- net DVDD renamed VDCDC
